File: EQD/Plumes/Plumes.kicad_sch (KiCad schematic)
At the start: 44 parts, among them J1 Conn_01x05_Pin, SW1 On-Off-On, U1 TL074, U2 LTC1044

Commit message: fix: 本家に倣って電解コンを使用
Parts:
- C13: footprint Capacitor_THT:C_Rect_L7.0mm_W6.5mm_P5.00mm -> Capacitor_THT:CP_Radial_D5.0mm_P2.00mm
Changed lines of the file:
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@@
 			)
 		)
-		(property "Footprint" "Capacitor_THT:C_Rect_L7.0mm_W6.5mm_P5.00mm"
+		(property "Footprint" "Capacitor_THT:CP_Radial_D5.0mm_P2.00mm"
 			(at 245.11 113.3348 0)
 			(hide yes)

Commit message: feat: コネクタピンを追加
Parts:
- removed J1: Conn_01x05_Pin, Connector_PinHeader_2.54mm:PinHeader_1x05_P2.54mm_Vertical, symbol Connector:Conn_01x05_Pin
- added J1: I/O, Connector_PinHeader_2.54mm:PinHeader_1x03_P2.54mm_Vertical, symbol Connector:Conn_01x03_Pin
- added J2: Power, Connector_PinHeader_2.54mm:PinHeader_1x02_P2.54mm_Vertical, symbol Connector:Conn_01x02_Pin
- added J3: LED, Connector_PinHeader_2.54mm:PinHeader_1x02_P2.54mm_Vertical, symbol Connector:Conn_01x02_Pin
- C1, C6: footprint Capacitor_THT:C_Rect_L7.2mm_W5.0mm_P5.00mm -> Capacitor_THT:C_Rect_L7.2mm_W4.5mm_P5.00mm_FKS2_FKP2_MKS2_MKP2
Connections:
- net +9V: now also J2.1 (Pin_1)
- net GND: now also J1.3 (Pin_3), J2.2 (Pin_2), J3.2 (Pin_2)
- net INPUT: now also J1.1 (Pin_1)
- net LED: now also J3.1 (Pin_1)
- net OUTPUT: now also J1.2 (Pin_2)

Commit message: feat: WIMAモデルのフットプリントを使用
Parts:
- C3: footprint Capacitor_THT:C_Rect_L13.0mm_W6.0mm_P10.00mm_FKS3_FKP3_MKS4 -> Capacitor_THT:C_Rect_L10.3mm_W5.7mm_P7.50mm_MKS4
Changed lines of the file:
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@@
 			)
 		)
-		(property "Footprint" "Capacitor_THT:C_Rect_L13.0mm_W6.0mm_P10.00mm_FKS3_FKP3_MKS4"
+		(property "Footprint" "Capacitor_THT:C_Rect_L10.3mm_W5.7mm_P7.50mm_MKS4"
 			(at 99.06 75.2348 0)
 			(hide yes)
