File: Paul.C/Timmy/Timmy.kicad_sch (KiCad schematic)
At the start: 35 parts, among them J1 I/O, J2 Power, J3 LED, SW1 SW_DIP_x02, U1 NJM4559

Commit message: feat: フットプリントを紐づけ
Parts:
- C7: footprint (none) -> Capacitor_THT:C_Rect_L7.0mm_W6.5mm_P5.00mm
Changed lines of the file:
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@@
 			)
 		)
-		(property "Footprint" ""
+		(property "Footprint" "Capacitor_THT:C_Rect_L7.0mm_W6.5mm_P5.00mm"
 			(at 162.56 75.2348 0)
 			(hide yes)

Commit message: feat: ReLayout Paul.C/Timmy
Parts:
- removed J1: I/O, Connector_PinHeader_2.54mm:PinHeader_1x03_P2.54mm_Vertical, symbol Connector:Conn_01x03_Pin
- added J2: Power, Connector_PinHeader_2.54mm:PinHeader_1x02_P2.54mm_Vertical, symbol Connector:Conn_01x02_Pin
- added J5: INPUT, Connector_PinHeader_2.54mm:PinHeader_1x01_P2.54mm_Vertical, symbol Connector:Conn_01x01_Pin
- C4: value 100p -> 101
- RV4: value A50k -> A10k
- renumbered C6 to C5, C5 to C6, J2 to J3, J3 to J4
Connections:
- net GND: now also J2.2 (Pin_2)
- net INPUT: now also J5.1 (Pin_1)
- net OUTPUT: now also J2.1 (Pin_1)
- net at C1.1, RV1.2: now also RV1.3
- no-connect marks 1 -> 0
Other:
- moved on the sheet: C1, C2, C3, C4, C5, C6, C7, C8, D7, J3, J4, R1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

Commit message: fix: オペアンプのフットプリントを修正
Parts:
- U1: footprint Package_DIP:DIP-8_W10.16mm -> Package_DIP:DIP-8_W7.62mm
Changed lines of the file:
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@@
 			)
 		)
-		(property "Footprint" "Package_DIP:DIP-8_W10.16mm"
+		(property "Footprint" "Package_DIP:DIP-8_W7.62mm"
 			(at 130.81 76.2 0)
 			(hide yes)
@@
 			)
 		)
-		(property "Footprint" "Package_DIP:DIP-8_W10.16mm"
+		(property "Footprint" "Package_DIP:DIP-8_W7.62mm"
 			(at 137.16 36.83 0)
 			(hide yes)
@@
 			)
 		)
-		(property "Footprint" "Package_DIP:DIP-8_W10.16mm"
+		(property "Footprint" "Package_DIP:DIP-8_W7.62mm"
 			(at 67.31 82.55 0)
 			(hide yes)

Commit message: refactor: 見直しに伴う形式的な更新
Parts:
- renumbered J5 to J1
Changed lines of the file:
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@@
 	(wire
 		(pts
-			(xy 107.95 63.5) (xy 110.49 63.5)
-		)
-		(stroke
-			(width 0)
-			(type default)
-		)
-	)
-	(wire
-		(pts
 			(xy 80.01 50.8) (xy 82.55 50.8)
 		)
@@
 	(wire
 		(pts
-			(xy 107.95 66.04) (xy 107.95 63.5)
-		)
-		(stroke
-			(width 0)
-			(type default)
-		)
-	)
-	(wire
-		(pts
 			(xy 31.75 38.1) (xy 31.75 44.45)
 		)
@@
 	(wire
 		(pts
-			(xy 44.45 95.25) (xy 44.45 92.71)
+			(xy 156.21 24.13) (xy 161.29 24.13)
 		)
 		(stroke
@@
 	(wire
 		(pts
-			(xy 156.21 24.13) (xy 161.29 24.13)
+			(xy 25.4 82.55) (xy 31.75 82.55)
 		)
 		(stroke
@@
 	(wire
 		(pts
-			(xy 25.4 82.55) (xy 31.75 82.55)
+			(xy 139.7 76.2) (xy 142.24 76.2)
 		)
 		(stroke
@@
 	(wire
 		(pts
-			(xy 139.7 76.2) (xy 142.24 76.2)
+			(xy 95.25 76.2) (xy 95.25 82.55)
 		)
 		(stroke
@@
 	(wire
 		(pts
-			(xy 95.25 76.2) (xy 95.25 82.55)
+			(xy 107.95 63.5) (xy 110.49 63.5)
 		)
 		(stroke
@@
 	(wire
 		(pts
+			(xy 44.45 92.71) (xy 50.8 92.71)
+		)
+		(stroke
+			(width 0)
+			(type default)
+		)
+	)
+	(wire
+		(pts
 			(xy 67.31 50.8) (xy 69.85 50.8)
 		)
@@
 		(dnp no)
 		(fields_autoplaced yes)
-		(property "Reference" "#PWR019"
+		(property "Reference" "#PWR018"
 			(at 171.45 95.25 0)
 			(hide yes)
@@
 			(project "Timmy"
 				(path "/ca2fbd8c-12cd-4803-bf08-d3c56d1caaa4"
-					(reference "#PWR019")
+					(reference "#PWR018")
 					(unit 1)
 				)
@@
 	(symbol
 		(lib_id "power:NEUT")
-		(at 107.95 66.04 180)
+		(at 107.95 63.5 0)
 		(unit 1)
 		(body_style 1)
@@
 		(in_pos_files yes)
 		(dnp no)
-		(fields_autoplaced yes)
 		(property "Reference" "#PWR05"
-			(at 107.95 62.23 0)
+			(at 107.95 67.31 0)
 			(hide yes)
 			(show_name no)
@@
 		)
 		(property "Value" "NEUT"
-			(at 107.95 71.12 0)
+			(at 105.41 58.42 0)
 			(show_name no)
 			(do_not_autoplace no)
@@
 					(size 1.27 1.27)
 				)
+				(justify left)
 			)
 		)
 		(property "Footprint" ""
-			(at 107.95 66.04 0)
+			(at 107.95 63.5 0)
 			(hide yes)
 			(show_name no)
@@
 		)
 		(property "Datasheet" ""
-			(at 107.95 66.04 0)
+			(at 107.95 63.5 0)
 			(hide yes)
 			(show_name no)
@@
 		)
 		(property "Description" "Power symbol creates a global label with name \"NEUT\""
-			(at 107.95 66.04 0)
+			(at 107.95 63.5 0)
 			(hide yes)
 			(show_name no)
@@
 		(dnp no)
 		(fields_autoplaced yes)
-		(property "Reference" "J5"
+		(property "Reference" "J1"
 			(at 182.245 68.58 0)
 			(show_name no)
@@
 			(project "Timmy"
 				(path "/ca2fbd8c-12cd-4803-bf08-d3c56d1caaa4"
-					(reference "J5")
+					(reference "J1")
 					(unit 1)
 				)
@@
 	(symbol
 		(lib_id "power:NEUT")
-		(at 44.45 95.25 180)
+		(at 50.8 92.71 0)
 		(unit 1)
 		(body_style 1)
@@
 		(in_pos_files yes)
 		(dnp no)
-		(fields_autoplaced yes)
 		(property "Reference" "#PWR04"
-			(at 44.45 91.44 0)
+			(at 50.8 96.52 0)
 			(hide yes)
 			(show_name no)
@@
 		)
 		(property "Value" "NEUT"
-			(at 44.45 100.33 0)
+			(at 48.26 88.9 0)
 			(show_name no)
 			(do_not_autoplace no)
@@
 					(size 1.27 1.27)
 				)
+				(justify left)
 			)
 		)
 		(property "Footprint" ""
-			(at 44.45 95.25 0)
+			(at 50.8 92.71 0)
 			(hide yes)
 			(show_name no)
@@
 		)
 		(property "Datasheet" ""
-			(at 44.45 95.25 0)
+			(at 50.8 92.71 0)
 			(hide yes)
 			(show_name no)
@@
 		)
 		(property "Description" "Power symbol creates a global label with name \"NEUT\""
-			(at 44.45 95.25 0)
+			(at 50.8 92.71 0)
 			(hide yes)
 			(show_name no)
@@
 		(dnp no)
 		(fields_autoplaced yes)
-		(property "Reference" "#PWR017"
+		(property "Reference" "#PWR016"
 			(at 181.61 85.09 0)
 			(hide yes)
@@
 			(project "Timmy"
 				(path "/ca2fbd8c-12cd-4803-bf08-d3c56d1caaa4"
-					(reference "#PWR017")
+					(reference "#PWR016")
 					(unit 1)
 				)
@@
 		(dnp no)
 		(fields_autoplaced yes)
-		(property "Reference" "#PWR018"
+		(property "Reference" "#PWR017"
 			(at 171.45 87.63 0)
 			(hide yes)
@@
 			(project "Timmy"
 				(path "/ca2fbd8c-12cd-4803-bf08-d3c56d1caaa4"
-					(reference "#PWR018")
+					(reference "#PWR017")
 					(unit 1)
 				)
@@
 		(dnp no)
 		(fields_autoplaced yes)
-		(property "Reference" "#PWR016"
+		(property "Reference" "#PWR015"
 			(at 171.45 80.01 0)
 			(hide yes)
@@
 			(project "Timmy"
 				(path "/ca2fbd8c-12cd-4803-bf08-d3c56d1caaa4"
-					(reference "#PWR016")
+					(reference "#PWR015")
 					(unit 1)
 				)
