File: ProCo/RAT/RAT.kicad_pcb (KiCad board)
At the start: 2 copper layers, 50.8 x 37.5 mm, 40 parts, among them J1 I/O, J2 Power, J3 Power, Q1 2N5458, SW1 SW_SPDT, U1 LM308N

Commit message: refactor: 見直しに伴う形式的な更新
Parts:
- D1: value 4001 -> 1N4001
- R1: value 2M2 -> 1M
- R4: renamed from R5; value 2M2 -> 1M
- renumbered R4 to R3, R3 to R5
Changed lines of the file:
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@@
 			)
 		)
-		(property "Value" "2M2"
+		(property "Value" "1M"
 			(at 3.81 0 90)
 			(layer "F.SilkS")
@@
 		(descr "Resistor, Axial_DIN0207 series, Axial, Horizontal, pin pitch=7.62mm, 0.25W = 1/4W, length*diameter=6.3*2.5mm^2, http://cdn-reichelt.de/documents/datenblatt/B400/1_4W%23YAG.pdf")
 		(tags "Resistor Axial_DIN0207 series Axial Horizontal pin pitch 7.62mm 0.25W = 1/4W length 6.3mm diameter 2.5mm")
-		(property "Reference" "R3"
+		(property "Reference" "R5"
 			(at 3.81 -2.37 90)
 			(layer "F.SilkS")
@@
 		(sheetname "/")
 		(sheetfile "RAT.kicad_sch")
+		(units
+			(unit
+				(name "A")
+				(pins "1" "2")
+			)
+		)
 		(attr through_hole)
 		(duplicate_pad_numbers_are_jumpers no)
@@
 		(descr "Resistor, Axial_DIN0207 series, Axial, Horizontal, pin pitch=7.62mm, 0.25W = 1/4W, length*diameter=6.3*2.5mm^2, http://cdn-reichelt.de/documents/datenblatt/B400/1_4W%23YAG.pdf")
 		(tags "Resistor Axial_DIN0207 series Axial Horizontal pin pitch 7.62mm 0.25W = 1/4W length 6.3mm diameter 2.5mm")
-		(property "Reference" "R5"
+		(property "Reference" "R4"
 			(at 3.81 -2.37 90)
 			(layer "F.SilkS")
@@
 			)
 		)
-		(property "Value" "2M2"
+		(property "Value" "1M"
 			(at 3.81 0 90)
 			(layer "F.SilkS")
@@
 		(sheetname "/")
 		(sheetfile "RAT.kicad_sch")
+		(units
+			(unit
+				(name "A")
+				(pins "1" "2")
+			)
+		)
 		(attr through_hole)
 		(duplicate_pad_numbers_are_jumpers no)
@@
 		(descr "Resistor, Axial_DIN0207 series, Axial, Horizontal, pin pitch=7.62mm, 0.25W = 1/4W, length*diameter=6.3*2.5mm^2, http://cdn-reichelt.de/documents/datenblatt/B400/1_4W%23YAG.pdf")
 		(tags "Resistor Axial_DIN0207 series Axial Horizontal pin pitch 7.62mm 0.25W = 1/4W length 6.3mm diameter 2.5mm")
-		(property "Reference" "R4"
+		(property "Reference" "R3"
 			(at 3.81 -2.37 0)
 			(layer "F.SilkS")
@@
 			)
 		)
-		(property "Value" "4001"
+		(property "Value" "1N4001"
 			(at 4.445 0 0)
 			(layer "F.SilkS")
@@
 		(sheetname "/")
 		(sheetfile "RAT.kicad_sch")
+		(units
+			(unit
+				(name "A")
+				(pins "1" "3" "2")
+			)
+		)
 		(attr through_hole)
 		(duplicate_pad_numbers_are_jumpers no)
@@
 		(sheetname "/")
 		(sheetfile "RAT.kicad_sch")
+		(units
+			(unit
+				(name "A")
+				(pins "1" "3" "2")
+			)
+		)
 		(attr through_hole)
 		(duplicate_pad_numbers_are_jumpers no)
@@
 		(sheetname "/")
 		(sheetfile "RAT.kicad_sch")
+		(units
+			(unit
+				(name "A")
+				(pins "1" "3" "2")
+			)
+		)
 		(attr through_hole)
 		(duplicate_pad_numbers_are_jumpers no)
@@
 	)
 	(arc
-		(start 93.0675 71.15)
+		(start 92.3925 71.15)
 		(mid 92.73 71.010202)
-		(end 92.3925 71.15)
+		(end 93.0675 71.15)
 		(width 0.5)
 		(layer "B.Cu")
@@
 	)
 	(segment
-		(start 85.745 46.0475)
-		(end 83.215234 48.577265)
+		(start 83.215234 48.577265)
+		(end 85.745 46.0475)
 		(width 0.5)
 		(layer "F.Cu")
@@
 	)
 	(arc
-		(start 81.6575 49.2225)
+		(start 83.215234 48.577265)
 		(mid 82.500539 49.054808)
-		(end 83.215234 48.577265)
+		(end 81.6575 49.2225)
 		(width 0.5)
 		(layer "F.Cu")
@@
 	)
 	(arc
-		(start 81.390234 49.867734)
+		(start 81.6575 49.2225)
 		(mid 81.308301 49.455826)
-		(end 81.6575 49.2225)
+		(end 81.390234 49.867734)
 		(width 0.5)
 		(layer "F.Cu")
@@
 	)
 	(segment
-		(start 106.921837 55.603011)
-		(end 106.478162 56.046686)
+		(start 106.478162 56.046686)
+		(end 106.921837 55.603011)
 		(width 1)
 		(layer "F.Cu")
@@
 	)
 	(segment
-		(start 105.665 56.859848)
-		(end 106.478162 56.046686)
+		(start 106.478162 56.046686)
+		(end 105.665 56.859848)
 		(width 1)
 		(layer "F.Cu")
@@
 	)
 	(arc
-		(start 124.039944 60.745056)
+		(start 123.825 61.263976)
 		(mid 123.880862 60.983138)
-		(end 123.825 61.263976)
+		(end 124.039944 60.745056)
 		(width 0.5)
 		(layer "F.Cu")
@@
 	)
 	(arc
-		(start 117.495 51.390525)
+		(start 118.13 49.8575)
 		(mid 117.660031 50.560857)
-		(end 118.13 49.8575)
+		(end 117.495 51.390525)
 		(width 0.5)
 		(layer "F.Cu")
