File: Fulltone/OCD/OCD.kicad_sch (KiCad schematic)
At the start: 26 parts, among them Q1 2N7000, Q2 2N7000, SW1 SW_SPDT, U1 TL082

Commit message: feat: フットプリントを紐づけ
Parts:
- added C10, C9: 100u, Capacitor_THT:CP_Radial_D8.0mm_P3.50mm, symbol Device:C_Polarized
- added D1: 1N4001, Diode_THT:D_DO-41_SOD81_P7.62mm_Horizontal, symbol Diode:1N4001
- added D2: LED, LED_THT:LED_D5.0mm, symbol Device:LED
- added J1: I/O, Connector_PinHeader_2.54mm:PinHeader_1x03_P2.54mm_Vertical, symbol Connector:Conn_01x03_Pin
- added J2, J3: Power, Connector_PinHeader_2.54mm:PinHeader_1x02_P2.54mm_Vertical, symbol Connector:Conn_01x02_Pin
- added R12: 100R, Resistor_THT:R_Axial_DIN0207_L6.3mm_D2.5mm_P7.62mm_Horizontal, symbol Device:R
- added R13, R14, R15: 10k, Resistor_THT:R_Axial_DIN0207_L6.3mm_D2.5mm_P7.62mm_Horizontal, symbol Device:R
- added unit 3 of U1
- C1, C3, C4, C6, C8: footprint (none) -> Capacitor_THT:C_Rect_L7.2mm_W3.0mm_P5.00mm_FKS2_FKP2_MKS2_MKP2
- C2: footprint (none) -> Capacitor_THT:C_Rect_L7.2mm_W4.5mm_P5.00mm_FKS2_FKP2_MKS2_MKP2
- C5: footprint (none) -> Capacitor_THT:C_Rect_L10.3mm_W5.7mm_P7.50mm_MKS4
- C7: footprint (none) -> Capacitor_THT:CP_Radial_D5.0mm_P2.00mm
- Q1, Q2: footprint Package_TO_SOT_THT:TO-92_Inline -> Package_TO_SOT_THT:TO-92_Inline_Wide
- R1, R10, R11, R2, R3, R4, R5, R6, R7, R8, R9: footprint (none) -> Resistor_THT:R_Axial_DIN0207_L6.3mm_D2.5mm_P7.62mm_Horizontal
- RV1, RV2, RV3: footprint (none) -> Potentiometer_THT:Potentiometer_Omeg_PC16BU_Vertical
- SW1: footprint (none) -> Connector_PinHeader_2.54mm:PinHeader_1x03_P2.54mm_Vertical
- U1: footprint (none) -> Package_DIP:DIP-8_W7.62mm
Connections:
- net GND: now also C10.2, C9.2, D1.2 (A), J1.3 (Pin_3), J2.2 (Pin_2), J3.2 (Pin_2), R15.1, U1.4 (V-)
- net INPUT: now also J1.1 (Pin_1)
- net NEUT: now also C10.1, R14.2, R15.2
- net OUTPUT: now also J1.2 (Pin_2)
- new net: C9.1, R12.2, R14.1, U1.8 (V+)
- new net: D2.2 (A), R13.2
- new net +9V: D1.1 (K), J2.1 (Pin_1), R12.1, R13.1
- new net LED: D2.1 (K), J3.1 (Pin_1)
Other:
- title: (none) -> Fulltone - OCD v3
- moved on the sheet: C1, C2, C3, C4, C5, C6, C7, C8, R1, R10, R11, R2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

Commit message: feat: ReLayout Fulltone/OCD v3
Parts:
- removed J1: I/O, Connector_PinHeader_2.54mm:PinHeader_1x03_P2.54mm_Vertical, symbol Connector:Conn_01x03_Pin
- removed J3: Power, Connector_PinHeader_2.54mm:PinHeader_1x02_P2.54mm_Vertical, symbol Connector:Conn_01x02_Pin
- added J1: INPUT, Connector_PinHeader_2.54mm:PinHeader_1x02_P2.54mm_Vertical, symbol Connector:Conn_01x02_Pin
- added J4: LED, Connector_PinHeader_2.54mm:PinHeader_1x01_P2.54mm_Vertical, symbol Connector:Conn_01x01_Pin
- added J5: OUTPUT, Connector_PinHeader_2.54mm:PinHeader_1x02_P2.54mm_Vertical, symbol Connector:Conn_01x02_Pin
- C4: renamed from C3; value 220p -> 221
- C8: renamed from C6; value 220p -> 221
- J3: renamed from J2; value Power -> +9V
- renumbered C8 to C10, C9 to C3, C10 to C5, C4 to C6, C5 to C7, C7 to C9, R6 to R10, R7 to R11, R8 to R12, R9 to R13, R10 to R14, R11 to R15, R12 to R4, R13 to R5, R14 to R6, R15 to R7, R4 to R8, R5 to R9
Connections:
- net GND: now also RV2.1, J1.2 (Pin_2), J5.2 (Pin_2); no longer RV2.2, RV2.3
- net INPUT: now also J1.1 (Pin_1)
- net LED: now also J4.1 (Pin_1)
- net OUTPUT: now also J5.1 (Pin_1)
- net at C10.2: now also RV2.2, RV2.3; no longer RV2.1
- net at C10.1, R15.2, RV3.3: now also SW1.1 (A); no longer SW1.3 (C)
Other:
- moved on the sheet: J3

Commit message: fix: コンデンサの定数を修正
Parts:
- C10: value 102 -> 473
- renumbered J5 to J1, J1 to J2
Changed lines of the file:
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@@
 		(dnp no)
 		(fields_autoplaced yes)
-		(property "Reference" "#PWR012"
+		(property "Reference" "#PWR013"
 			(at 127 72.39 0)
 			(hide yes)
@@
 			(project "OCD"
 				(path "/ed285c7d-4c7b-4eec-b4aa-2657f85b1869"
-					(reference "#PWR012")
+					(reference "#PWR013")
 					(unit 1)
 				)
@@
 		(dnp no)
 		(fields_autoplaced yes)
-		(property "Reference" "#PWR013"
+		(property "Reference" "#PWR014"
 			(at 137.16 85.09 0)
 			(hide yes)
@@
 			(project "OCD"
 				(path "/ed285c7d-4c7b-4eec-b4aa-2657f85b1869"
-					(reference "#PWR013")
+					(reference "#PWR014")
 					(unit 1)
 				)
@@
 		(dnp no)
 		(fields_autoplaced yes)
-		(property "Reference" "#PWR015"
+		(property "Reference" "#PWR016"
 			(at 171.45 82.55 0)
 			(hide yes)
@@
 			(project "OCD"
 				(path "/ed285c7d-4c7b-4eec-b4aa-2657f85b1869"
-					(reference "#PWR015")
+					(reference "#PWR016")
 					(unit 1)
 				)
@@
 		(dnp no)
 		(fields_autoplaced yes)
-		(property "Reference" "#PWR016"
+		(property "Reference" "#PWR012"
 			(at 125.73 80.01 0)
 			(hide yes)
@@
 			(project "OCD"
 				(path "/ed285c7d-4c7b-4eec-b4aa-2657f85b1869"
-					(reference "#PWR016")
+					(reference "#PWR012")
 					(unit 1)
 				)
@@
 		(dnp no)
 		(fields_autoplaced yes)
-		(property "Reference" "#PWR014"
+		(property "Reference" "#PWR015"
 			(at 127 87.63 0)
 			(hide yes)
@@
 			(project "OCD"
 				(path "/ed285c7d-4c7b-4eec-b4aa-2657f85b1869"
-					(reference "#PWR014")
+					(reference "#PWR015")
 					(unit 1)
 				)
@@
 		(dnp no)
 		(fields_autoplaced yes)
-		(property "Reference" "J1"
+		(property "Reference" "J2"
 			(at 139.7 69.8499 0)
 			(show_name no)
@@
 			(project "OCD"
 				(path "/ed285c7d-4c7b-4eec-b4aa-2657f85b1869"
-					(reference "J1")
+					(reference "J2")
 					(unit 1)
 				)
@@
 		(dnp no)
 		(fields_autoplaced yes)
-		(property "Reference" "J5"
+		(property "Reference" "J1"
 			(at 138.43 77.4699 0)
 			(show_name no)
@@
 			(project "OCD"
 				(path "/ed285c7d-4c7b-4eec-b4aa-2657f85b1869"
-					(reference "J5")
+					(reference "J1")
 					(unit 1)
 				)
@@
 			)
 		)
-		(property "Value" "102"
+		(property "Value" "473"
 			(at 161.29 58.4199 0)
 			(show_name no)

Commit message: fix: 何らかの修正
Parts:
- renumbered J2 to J1, J1 to J2
Other:
- moved on the sheet: J2
Changed lines of the file:
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@@
 	)
 	(label "OUTPUT"
-		(at 132.08 77.47 180)
+		(at 133.35 77.47 180)
 		(effects
 			(font
@@
 		(dnp no)
 		(fields_autoplaced yes)
-		(property "Reference" "#PWR013"
+		(property "Reference" "#PWR012"
 			(at 127 72.39 0)
 			(hide yes)
@@
 			(project "OCD"
 				(path "/ed285c7d-4c7b-4eec-b4aa-2657f85b1869"
-					(reference "#PWR013")
+					(reference "#PWR012")
 					(unit 1)
 				)
@@
 	(symbol
 		(lib_id "power:GND")
-		(at 132.08 80.01 270)
+		(at 133.35 80.01 270)
 		(unit 1)
 		(body_style 1)
@@
 		(dnp no)
 		(fields_autoplaced yes)
-		(property "Reference" "#PWR012"
-			(at 125.73 80.01 0)
+		(property "Reference" "#PWR013"
+			(at 127 80.01 0)
 			(hide yes)
 			(show_name no)
@@
 		)
 		(property "Value" "GND"
-			(at 127 80.01 0)
+			(at 128.27 80.01 0)
 			(hide yes)
 			(show_name no)
@@
 		)
 		(property "Footprint" ""
-			(at 132.08 80.01 0)
+			(at 133.35 80.01 0)
 			(hide yes)
 			(show_name no)
@@
 		)
 		(property "Datasheet" ""
-			(at 132.08 80.01 0)
+			(at 133.35 80.01 0)
 			(hide yes)
 			(show_name no)
@@
 		)
 		(property "Description" "Power symbol creates a global label with name \"GND\" , ground"
-			(at 132.08 80.01 0)
+			(at 133.35 80.01 0)
 			(hide yes)
 			(show_name no)
@@
 			(project "OCD"
 				(path "/ed285c7d-4c7b-4eec-b4aa-2657f85b1869"
-					(reference "#PWR012")
+					(reference "#PWR013")
 					(unit 1)
 				)
@@
 		(dnp no)
 		(fields_autoplaced yes)
-		(property "Reference" "J2"
+		(property "Reference" "J1"
 			(at 139.7 69.8499 0)
 			(show_name no)
@@
 			(project "OCD"
 				(path "/ed285c7d-4c7b-4eec-b4aa-2657f85b1869"
-					(reference "J2")
+					(reference "J1")
 					(unit 1)
 				)
@@
 	(symbol
 		(lib_id "Connector:Conn_01x02_Pin")
-		(at 137.16 77.47 0)
+		(at 138.43 77.47 0)
 		(mirror y)
 		(unit 1)
@@
 		(dnp no)
 		(fields_autoplaced yes)
-		(property "Reference" "J1"
-			(at 138.43 77.4699 0)
+		(property "Reference" "J2"
+			(at 139.7 77.4699 0)
 			(show_name no)
 			(do_not_autoplace no)
@@
 		)
 		(property "Value" "OUTPUT"
-			(at 138.43 80.0099 0)
+			(at 139.7 80.0099 0)
 			(show_name no)
 			(do_not_autoplace no)
@@
 		)
 		(property "Footprint" "Connector_PinHeader_2.54mm:PinHeader_1x02_P2.54mm_Vertical"
-			(at 137.16 77.47 0)
+			(at 138.43 77.47 0)
 			(hide yes)
 			(show_name no)
@@
 		)
 		(property "Datasheet" ""
-			(at 137.16 77.47 0)
+			(at 138.43 77.47 0)
 			(hide yes)
 			(show_name no)
@@
 		)
 		(property "Description" "Generic connector, single row, 01x02, script generated"
-			(at 137.16 77.47 0)
+			(at 138.43 77.47 0)
 			(hide yes)
 			(show_name no)
@@
 			(project "OCD"
 				(path "/ed285c7d-4c7b-4eec-b4aa-2657f85b1869"
-					(reference "J1")
+					(reference "J2")
 					(unit 1)
 				)
