File: EHX/BIG MUFF [Triangle]/BIG MUFF [Triangle].kicad_pcb (KiCad board)
At the start: 2 copper layers, 55.9 x 46.4 mm, 55 parts, among them J1 INPUT, J2 Power, J3 LED, J4 OUTPUT, Q1 2N3904, Q2 2N3904, Q3 2N3904, Q4 2N3904

Commit message: refactor: 見直しに伴う形式的な更新
Parts:
- C11: value 392 -> 402
- renumbered J4 to J2, J2 to J3, J3 to J4
Changed lines of the file:
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@@
 		(descr "Through hole straight pin header, 1x02, 2.54mm pitch, single row")
 		(tags "Through hole pin header THT 1x02 2.54mm single row")
-		(property "Reference" "J3"
+		(property "Reference" "J4"
 			(at 0 -2.38 90)
 			(layer "F.SilkS")
@@
 			)
 		)
-		(property "Value" "392"
+		(property "Value" "402"
 			(at 2.5 0 90)
 			(layer "F.SilkS")
@@
 		(descr "Through hole straight pin header, 1x02, 2.54mm pitch, single row")
 		(tags "Through hole pin header THT 1x02 2.54mm single row")
-		(property "Reference" "J2"
+		(property "Reference" "J3"
 			(at 0 -2.38 90)
 			(layer "F.SilkS")
@@
 		(descr "Through hole straight pin header, 1x01, 2.54mm pitch, single row")
 		(tags "Through hole pin header THT 1x01 2.54mm single row")
-		(property "Reference" "J4"
+		(property "Reference" "J2"
 			(at 0 -2.38 0)
 			(layer "F.SilkS")

Commit message: fix: 1N4148のフットプリントが小さすぎた
Parts:
- removed D3, D4, D5, D6: 1N4148, Diode_THT:D_DO-35_SOD27_P3.81mm_Vertical_AnodeUp
- added D10: 1N4148, Diode_THT:D_DO-35_SOD27_P5.08mm_Vertical_AnodeUp, F.Cu at (121.1, 96.5)
- added D7: 1N4148, Diode_THT:D_DO-35_SOD27_P5.08mm_Vertical_AnodeUp, F.Cu at (144.1, 78.7)
- added D8: 1N4148, Diode_THT:D_DO-35_SOD27_P5.08mm_Vertical_AnodeUp, F.Cu at (149.2, 81.3)
- added D9: 1N4148, Diode_THT:D_DO-35_SOD27_P5.08mm_Vertical_AnodeUp, F.Cu at (116.1, 99.1)
- C10, C2, C7: value 500p -> 501
- RV1: value B100k -> B00k
- moved C7 0.79 mm to (152.4, 83.8)
- moved C6 0.48 mm to (141.0, 78.8)
Routing:
- net Net-(Q2-B): track 26.8 -> 24.6 mm
- net Net-(D10-K): track 54.2 -> 52.2 mm
- net Net-(D7-A): track 30.8 -> 28.9 mm
- net GND: vias 72 -> 89
Other:
- board text added: "EHX - BIG MUFF [Triangle] [ReLayouted] 2026/08/18"
