File: EHX/BIG MUFF [Russian]/BIG MUFF [Russian].kicad_pcb (KiCad board)
At the start: 2 copper layers, 55.9 x 46.4 mm, 55 parts, among them J1 INPUT, J2 Power, J3 LED, J4 OUTPUT, Q1 2N3904, Q2 2N3904, Q3 2N3904, Q4 2N3904

Commit message: fix: GNDビアを追加
Routing:
- net GND: vias 66 -> 72
Other:
- board text added: "EHX - BIG MUFF [Russian] [ReLayouted] 2026/08/18"
Changed lines of the file:
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@@
+		)
+	)
+	(gr_text "EHX - BIG MUFF [Russian]\n[ReLayouted] 2026/08/18"
+		(at 152.4 71.12 0)
+		(layer "B.SilkS")
+		(effects
+			(font
+				(size 1 1)
+				(bold yes)
+			)
+			(justify mirror)
 		)
 	)
@@
 	)
 	(via
+		(at 158.75 83.185)
+		(size 0.6)
+		(drill 0.3)
+		(layers "F.Cu" "B.Cu")
+		(free yes)
+		(net "GND")
+	)
+	(via
 		(at 158.75 56.515)
 		(size 0.6)
@@
 	)
 	(via
+		(at 151.13 99.695)
+		(size 0.6)
+		(drill 0.3)
+		(layers "F.Cu" "B.Cu")
+		(free yes)
+		(net "GND")
+	)
+	(via
 		(at 138.43 95.25)
 		(size 0.6)
@@
 	)
 	(via
+		(at 161.925 83.185)
+		(size 0.6)
+		(drill 0.3)
+		(layers "F.Cu" "B.Cu")
+		(free yes)
+		(net "GND")
+	)
+	(via
 		(at 142.24 96.52)
 		(size 0.6)
@@
 	)
 	(via
+		(at 153.67 99.695)
+		(size 0.6)
+		(drill 0.3)
+		(layers "F.Cu" "B.Cu")
+		(free yes)
+		(net "GND")
+	)
+	(via
 		(at 142.24 73.025)
 		(size 0.6)
@@
 	)
 	(via
+		(at 155.575 83.185)
+		(size 0.6)
+		(drill 0.3)
+		(layers "F.Cu" "B.Cu")
+		(free yes)
+		(net "GND")
+	)
+	(via
 		(at 142.24 71.12)
 		(size 0.6)
@@
 		(size 0.6)
 		(drill 0.3)
+		(layers "F.Cu" "B.Cu")
+		(free yes)
+		(net "GND")
+	)
+	(via
+		(at 148.59 99.695)
+		(size 0.6)
+		(drill 0.3)

Commit message: refactor: 見直しに伴う形式的な更新
Parts:
- renumbered J4 to J2, J2 to J3, J3 to J4
Changed lines of the file:
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@@
 		(sheetname "/")
 		(sheetfile "BIG MUFF [Russian].kicad_sch")
+		(units
+			(unit
+				(name "A")
+				(pins "1" "2")
+			)
+		)
 		(attr through_hole)
 		(duplicate_pad_numbers_are_jumpers no)
@@
 		(descr "Through hole straight pin header, 1x02, 2.54mm pitch, single row")
 		(tags "Through hole pin header THT 1x02 2.54mm single row")
-		(property "Reference" "J3"
+		(property "Reference" "J4"
 			(at 0 -2.38 90)
 			(layer "F.SilkS")
@@
 		(descr "Through hole straight pin header, 1x02, 2.54mm pitch, single row")
 		(tags "Through hole pin header THT 1x02 2.54mm single row")
-		(property "Reference" "J2"
+		(property "Reference" "J3"
 			(at 0 -2.38 90)
 			(layer "F.SilkS")
@@
 		(descr "Through hole straight pin header, 1x01, 2.54mm pitch, single row")
 		(tags "Through hole pin header THT 1x01 2.54mm single row")
-		(property "Reference" "J4"
+		(property "Reference" "J2"
 			(at 0 -2.38 0)
 			(layer "F.SilkS")
@@
 		(sheetname "/")
 		(sheetfile "BIG MUFF [Russian].kicad_sch")
+		(units
+			(unit
+				(name "A")
+				(pins "1" "2")
+			)
+		)
 		(attr through_hole)
 		(duplicate_pad_numbers_are_jumpers no)

Commit message: fix: 1N4148のフットプリントが小さすぎた
Parts:
- removed D3, D4, D5, D6: 1N4148, Diode_THT:D_DO-35_SOD27_P3.81mm_Vertical_AnodeUp
- added D10: 1N4148, Diode_THT:D_DO-35_SOD27_P5.08mm_Vertical_AnodeUp, F.Cu at (121.1, 96.5)
- added D7: 1N4148, Diode_THT:D_DO-35_SOD27_P5.08mm_Vertical_AnodeUp, F.Cu at (144.1, 78.7)
- added D8: 1N4148, Diode_THT:D_DO-35_SOD27_P5.08mm_Vertical_AnodeUp, F.Cu at (149.2, 81.3)
- added D9: 1N4148, Diode_THT:D_DO-35_SOD27_P5.08mm_Vertical_AnodeUp, F.Cu at (116.1, 99.1)
- C10, C7: value 470p -> 471
- moved C7 0.79 mm to (152.4, 83.8)
- moved C6 0.48 mm to (141.0, 78.8)
Routing:
- net Net-(Q2-B): track 26.8 -> 24.6 mm
- net Net-(D10-K): track 54.2 -> 52.2 mm
- net Net-(D7-A): track 30.8 -> 28.9 mm
- net GND: vias 72 -> 89

Commit message: fix: 数値の向きを修正
Parts:
- C2: value 470p -> 471
Changed lines of the file:
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@@
 			)
 		)
-		(property "Value" "470p"
-			(at 2.5 0 180)
+		(property "Value" "471"
+			(at 2.5 0 270)
 			(layer "F.SilkS")
 			(effects
